Commit message: today

File: gr00t_wbc/control/robot_model/model_data/g1/g1_29dof_with_hand.urdf (robot description, URDF)
Before this commit: robot g1_29dof_with_hand, 53 links, 52 joints
Links:
- added link right_hand_palm_center
Joints:
- added joint right_hand_palm_center_joint: type fixed, parent right_hand_palm_link, child right_hand_palm_center, origin xyz=0.01214634836 0.00050869656 -0.00058171093 rpy=0 0 0

Commit message: rotate waist

File: gr00t_wbc/control/robot_model/model_data/g1/g1_29dof_with_hand.urdf (robot description, URDF)
Before this commit: robot g1_29dof_with_hand, 54 links, 53 joints
Links:
- added link right_hand_grip_center
Joints:
- added joint right_hand_grip_center_joint: type fixed, parent right_hand_palm_center, child right_hand_grip_center, origin xyz=0.085 0.07 0.03 rpy=0 0 0

Commit message: grabbing adjustments

File: gr00t_wbc/control/robot_model/model_data/g1/g1_29dof_with_hand.urdf (robot description, URDF)
Before this commit: robot g1_29dof_with_hand, 55 links, 54 joints
Links:
- added link left_hand_grip_center
- added link left_hand_palm_center
Joints:
- added joint left_hand_grip_center_joint: type fixed, parent left_hand_palm_center, child left_hand_grip_center, origin xyz=0.049 -0.09 0.025 rpy=0 0 0
- added joint left_hand_palm_center_joint: type fixed, parent left_hand_palm_link, child left_hand_palm_center, origin xyz=0.01214634836 -0.00050869656 -0.00058171093 rpy=0 0 0
- joint right_hand_grip_center_joint: origin xyz=0.085 0.07 0.03 rpy=0 0 0 -> xyz=0.049 0.09 0.025 rpy=0 0 0
